File: Hardware/SparkFun_Thing_Plus_NINA-B306.sch (EAGLE design)
At the start: 82 parts, among them J1 USB-C, J2 THING_PLUS_LOGICAL, J3 CONN_03X2, J4 MICRO-SDFRICTION, J6 QWIIC_RA, Q1 20V/4.2A/52mΩ/1.4W, Q2 220mA/50V/3.5Ω, Q3 20V/4.2A/52mΩ/1.4W, U1 ESD Diode, U2 U-BLOX_NINA_B306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

Commit message: Updates in prep for sch review
Schematic: Replaced 0603 10ks with 0402T package.

Board: Initial layout of parts complete.
Parts:
- R11, R12, R14, R15, R16: device SparkFun-Resistors:10KOHM-0603-1/10W-1% -> SparkFun-Resistors:10KOHM-0402T-1/16W-1%
Changed lines of the file:
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@@
 <part name="SUPPLY11" library="SparkFun-PowerSymbols" deviceset="3.3V" device=""/>
 <part name="GND14" library="SparkFun-PowerSymbols" deviceset="GND" device=""/>
-<part name="R11" library="SparkFun-Resistors" deviceset="10KOHM" device="-0603-1/10W-1%" value="10k"/>
-<part name="R12" library="SparkFun-Resistors" deviceset="10KOHM" device="-0603-1/10W-1%" value="10k"/>
+<part name="R11" library="SparkFun-Resistors" deviceset="10KOHM" device="-0402T-1/16W-1%" value="10k"/>
+<part name="R12" library="SparkFun-Resistors" deviceset="10KOHM" device="-0402T-1/16W-1%" value="10k"/>
 <part name="GND18" library="SparkFun-PowerSymbols" deviceset="GND" device=""/>
 <part name="Q2" library="SparkFun-DiscreteSemi" deviceset="MOSFET-NCH" device="-BSS138" value="220mA/50V/3.5Ω"/>
@@
 <part name="SUPPLY28" library="SparkFun-PowerSymbols" deviceset="3.3V" device=""/>
 <part name="SUPPLY29" library="SparkFun-PowerSymbols" deviceset="3.3V" device=""/>
-<part name="R15" library="SparkFun-Resistors" deviceset="10KOHM" device="-0603-1/10W-1%" value="10k"/>
+<part name="R15" library="SparkFun-Resistors" deviceset="10KOHM" device="-0402T-1/16W-1%" value="10k"/>
 <part name="SUPPLY30" library="SparkFun-PowerSymbols" deviceset="3.3V" device=""/>
 <part name="GND38" library="SparkFun-PowerSymbols" deviceset="GND" device=""/>
 <part name="U6" library="SparkFun-Sensors" deviceset="ISM330DHCX" device=""/>
-<part name="R14" library="SparkFun-Resistors" deviceset="10KOHM" device="-0603-1/10W-1%" value="10k"/>
+<part name="R14" library="SparkFun-Resistors" deviceset="10KOHM" device="-0402T-1/16W-1%" value="10k"/>
 <part name="SUPPLY31" library="SparkFun-PowerSymbols" deviceset="3.3V" device=""/>
-<part name="R16" library="SparkFun-Resistors" deviceset="10KOHM" device="-0603-1/10W-1%" value="10k"/>
+<part name="R16" library="SparkFun-Resistors" deviceset="10KOHM" device="-0402T-1/16W-1%" value="10k"/>
 <part name="SUPPLY32" library="SparkFun-PowerSymbols" deviceset="3.3V" device=""/>
 <part name="GND39" library="SparkFun-PowerSymbols" deviceset="GND" device=""/>

Commit message: Changed package of 100R, rearrange board.
Changed 100R from 0603 to 0402T and rearranged the board to better organize that circuit. Also moved the QWIIC logo next to the QWIIC connector with the new space.
Parts:
- R13: device SparkFun-Resistors:100OHM-0603-1/10W-1% -> SparkFun-Resistors:100OHM-0402-TIGHT-1/16W-1%
Changed lines of the file:
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@@
 <part name="GND18" library="SparkFun-PowerSymbols" deviceset="GND" device=""/>
 <part name="Q2" library="SparkFun-DiscreteSemi" deviceset="MOSFET-NCH" device="-BSS138" value="220mA/50V/3.5Ω"/>
-<part name="R13" library="SparkFun-Resistors" deviceset="100OHM" device="-0603-1/10W-1%" value="100"/>
+<part name="R13" library="SparkFun-Resistors" deviceset="100OHM" device="-0402-TIGHT-1/16W-1%" value="100"/>
 <part name="SUPPLY14" library="SparkFun-PowerSymbols" deviceset="3.3V" device=""/>
 <part name="SUPPLY24" library="SparkFun-PowerSymbols" deviceset="3.3V" device=""/>

Commit message: Added net classing, net names.
Connections:
- net N$17 renamed SCL_PU_PWR
- net N$7 renamed 3V3_QWIIC
- net N$9 renamed SDA_PU_PWR
Changed lines of the file:
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@@
 </variantdefs>
 <classes>
-<class number="0" name="default" width="0" drill="0">
+<class number="0" name="default" width="0.11" drill="0.3">
+<clearance class="0" value="0.11"/>
 </class>
-<class number="1" name="power" width="0.3048" drill="0.3048">
+<class number="1" name="power" width="0.2" drill="0.3">
+<clearance class="1" value="0.3"/>
+</class>
+<class number="2" name="ground" width="0.11" drill="0.3">
+<clearance class="0" value="0.2"/>
+<clearance class="1" value="0.11"/>
+</class>
+<class number="3" name="analog" width="0.2" drill="0.3">
+<clearance class="0" value="0.3"/>
+<clearance class="1" value="0.3"/>
+<clearance class="2" value="0.2"/>
+<clearance class="3" value="0.2"/>
+</class>
+<class number="4" name="HS_digital" width="0.11" drill="0.3">
+<clearance class="0" value="0.2"/>
+<clearance class="1" value="0.3"/>
+<clearance class="2" value="0.2"/>
+<clearance class="3" value="1"/>
+<clearance class="4" value="0.15"/>
+</class>
+<class number="5" name="usb_diff" width="0.24" drill="0.3">
+<clearance class="0" value="0.4"/>
+<clearance class="1" value="0.23"/>
+<clearance class="2" value="0.4"/>
+<clearance class="3" value="1"/>
+<clearance class="4" value="0.4"/>
+<clearance class="5" value="0.23"/>
 </class>
 </classes>
@@
 </busses>
 <nets>
-<net name="GND" class="0">
+<net name="GND" class="2">
 <segment>
 <pinref part="GND1" gate="1" pin="GND"/>
@@
 </segment>
 </net>
-<net name="USB_N" class="0">
+<net name="USB_N" class="5">
 <segment>
 <pinref part="J1" gate="J1" pin="D-"/>
@@
 </segment>
 </net>
-<net name="USB_P" class="0">
+<net name="USB_P" class="5">
 <segment>
 <pinref part="J1" gate="J1" pin="D+"/>
@@
 </segment>
 </net>
-<net name="V_USB" class="0">
+<net name="V_USB" class="1">
 <segment>
 <pinref part="SUPPLY1" gate="G$1" pin="V_USB"/>
@@
 </segment>
 </net>
-<net name="V_BATT" class="0">
+<net name="V_BATT" class="1">
 <segment>
 <pinref part="U4" gate="G$1" pin="VBAT"/>
@@
 </segment>
 </net>
-<net name="VIN" class="0">
+<net name="VIN" class="1">
 <segment>
 <pinref part="D3" gate="G$1" pin="C"/>
@@
 </segment>
 </net>
-<net name="3.3V" class="0">
+<net name="3.3V" class="1">
 <segment>
 <pinref part="C8" gate="G$1" pin="1"/>
@@
 </segment>
 </net>
-<net name="IO48/POCI" class="0">
+<net name="IO48/POCI" class="4">
 <segment>
 <wire x1="281.94" y1="30.48" x2="279.4" y2="30.48" width="0.1524" layer="91"/>
@@
 </segment>
 </net>
-<net name="IO50/PICO" class="0">
+<net name="IO50/PICO" class="4">
 <segment>
 <wire x1="281.94" y1="25.4" x2="279.4" y2="25.4" width="0.1524" layer="91"/>
@@
 </segment>
 </net>
-<net name="IO52/SCK" class="0">
+<net name="IO52/SCK" class="4">
 <segment>
 <wire x1="281.94" y1="27.94" x2="279.4" y2="27.94" width="0.1524" layer="91"/>
@@
 </segment>
 </net>
-<net name="SWCLK" class="0">
+<net name="SWCLK" class="4">
 <segment>
 <wire x1="213.36" y1="30.48" x2="215.9" y2="30.48" width="0.1524" layer="91"/>
@@
 </segment>
 </net>
-<net name="SWDIO" class="0">
+<net name="SWDIO" class="4">
 <segment>
 <wire x1="233.68" y1="33.02" x2="231.14" y2="33.02" width="0.1524" layer="91"/>
@@
 </segment>
 </net>
-<net name="IO20/A3" class="0">
+<net name="IO20/A3" class="3">
 <segment>
 <wire x1="109.22" y1="137.16" x2="106.68" y2="137.16" width="0.1524" layer="91"/>
@@
 </segment>
 </net>
-<net name="IO24/A0" class="0">
+<net name="IO24/A0" class="3">
 <segment>
 <wire x1="109.22" y1="127" x2="106.68" y2="127" width="0.1524" layer="91"/>
@@
 </segment>
 </net>
-<net name="IO23/A1" class="0">
+<net name="IO23/A1" class="3">
 <segment>
 <wire x1="109.22" y1="129.54" x2="106.68" y2="129.54" width="0.1524" layer="91"/>
@@
 </segment>
 </net>
-<net name="IO27/A2" class="0">
+<net name="IO27/A2" class="3">
 <segment>
 <wire x1="109.22" y1="121.92" x2="106.68" y2="121.92" width="0.1524" layer="91"/>
@@
 </segment>
 </net>
-<net name="IO17/A5" class="0">
+<net name="IO17/A5" class="3">
 <segment>
 <wire x1="109.22" y1="142.24" x2="106.68" y2="142.24" width="0.1524" layer="91"/>
@@
 </segment>
 </net>
-<net name="IO18/A4" class="0">
+<net name="IO18/A4" class="3">
 <segment>
 <wire x1="109.22" y1="139.7" x2="106.68" y2="139.7" width="0.1524" layer="91"/>
@@
 </segment>
 </net>
-<net name="IO42/SCL" class="0">
+<net name="IO42/SCL" class="4">
 <segment>
 <pinref part="U2" gate="G$1" pin="IO42"/>
@@
 </segment>
 </net>
-<net name="IO43/SDA" class="0">
+<net name="IO43/SDA" class="4">
 <segment>
 <pinref part="U2" gate="G$1" pin="IO43"/>
@@
 </segment>
 </net>
-<net name="IO7/NINA_TX/DEV_RX" class="0">
+<net name="IO7/NINA_TX/DEV_RX" class="4">
 <segment>
 <pinref part="U2" gate="G$1" pin="IO7"/>
@@
 </segment>
 </net>
-<net name="IO5/NINA_RX/DEV_TX" class="0">
+<net name="IO5/NINA_RX/DEV_TX" class="4">
 <segment>
 <pinref part="U2" gate="G$1" pin="IO5"/>
@@
 </segment>
 </net>
-<net name="N$9" class="0">
+<net name="SDA_PU_PWR" class="1">
 <segment>
 <pinref part="R7" gate="G$1" pin="2"/>
@@
 </segment>
 </net>
-<net name="N$17" class="0">
+<net name="SCL_PU_PWR" class="1">
 <segment>
 <pinref part="R5" gate="G$1" pin="2"/>
@@
 </segment>
 </net>
-<net name="N$7" class="0">
+<net name="3V3_QWIIC" class="1">
 <segment>
 <pinref part="Q3" gate="G$1" pin="D"/>
@@
 </segment>
 </net>
-<net name="N$12" class="0">
-<segment>
-<wire x1="287.02" y1="139.7" x2="287.02" y2="137.16" width="0.1524" layer="91"/>
-<wire x1="287.02" y1="137.16" x2="292.1" y2="137.16" width="0.1524" layer="91"/>
-<wire x1="292.1" y1="137.16" x2="292.1" y2="134.62" width="0.1524" layer="91"/>
-<pinref part="R12" gate="G$1" pin="1"/>
-<pinref part="R13" gate="G$1" pin="2"/>
-<pinref part="Q3" gate="G$1" pin="G"/>
-<wire x1="292.1" y1="144.78" x2="292.1" y2="137.16" width="0.1524" layer="91"/>
-<junction x="292.1" y="137.16"/>
-</segment>
-</net>
 <net name="N$13" class="0">
 <segment>
@@
 </segment>
 </net>
+<net name="N$7" class="0">
+<segment>
+<pinref part="R12" gate="G$1" pin="1"/>
+<wire x1="292.1" y1="137.16" x2="287.02" y2="137.16" width="0.1524" layer="91"/>
+<wire x1="287.02" y1="137.16" x2="287.02" y2="139.7" width="0.1524" layer="91"/>
+<pinref part="Q3" gate="G$1" pin="G"/>
+<wire x1="292.1" y1="144.78" x2="292.1" y2="137.16" width="0.1524" layer="91"/>
+<pinref part="R13" gate="G$1" pin="2"/>
+<wire x1="292.1" y1="134.62" x2="292.1" y2="137.16" width="0.1524" layer="91"/>
+<junction x="292.1" y="137.16"/>
+</segment>
+</net>
