File: Hardware/SparkFun_Thing_Plus_NINA-B306.brd (EAGLE design)
At the start: 22.9 x 66 mm, 84 parts, among them J1 USB-C, J2 THING_PLUS_LOGICAL, J3 CONN_03X2, J4 MICRO-SDFRICTION, J6 QWIIC_RA, Q1 20V/4.2A/52mΩ/1.4W, Q2 220mA/50V/3.5Ω, Q3 20V/4.2A/52mΩ/1.4W, U1 ESD Diode, U2 U-BLOX_NINA_B306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

Commit message: Routed high speed and analog.
Parts:
- moved J3 11.9 mm to (13.5, 60.2)
- moved C2 0.40 mm to (18.6, 61.5)
- moved C3 0.40 mm to (18.6, 60.5)
Routing:
- net IO48/POCI: track 0.00 -> 53.3 mm, vias 0 -> 2
- net IO52/SCK: track 0.00 -> 52.4 mm, vias 0 -> 2
- net IO50/PICO: track 0.00 -> 50.8 mm, vias 0 -> 2
- net IO24/A0: track 0.00 -> 38.3 mm, vias 0 -> 1
- net IO23/A1: track 0.00 -> 36.8 mm, vias 0 -> 1
- net IO20/A3: track 0.00 -> 34.3 mm, vias 0 -> 1
- net IO18/A4: track 0.00 -> 33.2 mm, vias 0 -> 1
- net IO17/A5: track 0.00 -> 31.8 mm, vias 0 -> 1
- net IO27/A2: track 0.00 -> 31.0 mm, vias 0 -> 1
- net IO7/NINA_TX/DEV_RX: track 0.00 -> 13.0 mm
- net IO5/NINA_RX/DEV_TX: track 0.00 -> 12.7 mm
- net SWDIO: track 0.00 -> 3.30 mm, vias 0 -> 1
- net SWCLK: track 0.00 -> 2.78 mm, vias 0 -> 1

Commit message: Routing, end of week commit.
Parts:
- J3: value CONN_03X2 -> CONN_03X2_NO4; device MISC:PAD_05_03X2_TP -> MISC:PAD_05_03X2_TP_NO4
- moved U1 0.40 mm to (16.1, 9.50)
Routing:
- net USB_P: track 0.00 -> 9.96 mm, vias 0 -> 2
- net USB_N: track 0.00 -> 9.70 mm
- net !RESET!: track 0.00 -> 7.59 mm
